File: _autosave-ubox_with_stm32.kicad_sch (KiCad schematic)
At the start: 22 parts, among them J1 I2c_pin, J3 UART_Pin, U3 SAM-M10Q-00B

Commit message: resize component
Parts:
- C2: footprint Capacitor_SMD:C_0201_0603Metric -> Capacitor_SMD:C_0805_2012Metric
- D2, D3: footprint LED_SMD:LED_0402_1005Metric -> LED_SMD:LED_0805_2012Metric
Changed lines of the file:
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@@
 			)
 		)
-		(property "Footprint" "Capacitor_SMD:C_0201_0603Metric"
+		(property "Footprint" "Capacitor_SMD:C_0805_2012Metric"
 			(at 100.0252 60.96 0)
 			(effects
@@
 			)
 		)
-		(property "Footprint" "LED_SMD:LED_0402_1005Metric"
+		(property "Footprint" "LED_SMD:LED_0805_2012Metric"
 			(at 29.21 135.89 0)
 			(effects
@@
 			)
 		)
-		(property "Footprint" "LED_SMD:LED_0402_1005Metric"
+		(property "Footprint" "LED_SMD:LED_0805_2012Metric"
 			(at 54.61 135.89 0)
 			(effects

Commit message: compatible with breadboard
Parts:
- J1, J3: footprint Connector_PinHeader_1.00mm:PinHeader_1x04_P1.00mm_Horizontal -> Connector_PinHeader_1.00mm:PinHeader_1x04_P1.00mm_Vertical
- J2: footprint Connector_PinHeader_1.00mm:PinHeader_1x06_P1.00mm_Horizontal -> Connector_PinHeader_1.00mm:PinHeader_1x06_P1.00mm_Vertical
Changed lines of the file:
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@@
 			)
 		)
-		(property "Footprint" "Connector_PinHeader_1.00mm:PinHeader_1x06_P1.00mm_Horizontal"
+		(property "Footprint" "Connector_PinHeader_1.00mm:PinHeader_1x06_P1.00mm_Vertical"
 			(at 139.7 143.51 0)
 			(effects
@@
 			)
 		)
-		(property "Footprint" "Connector_PinHeader_1.00mm:PinHeader_1x04_P1.00mm_Horizontal"
+		(property "Footprint" "Connector_PinHeader_1.00mm:PinHeader_1x04_P1.00mm_Vertical"
 			(at 176.53 114.3 0)
 			(effects
@@
 			)
 		)
-		(property "Footprint" "Connector_PinHeader_1.00mm:PinHeader_1x04_P1.00mm_Horizontal"
+		(property "Footprint" "Connector_PinHeader_1.00mm:PinHeader_1x04_P1.00mm_Vertical"
 			(at 139.7 114.3 0)
 			(effects
